File: hardware/kicad/kc2_left-x3/kc2_left-x3.kicad_pcb (KiCad board)
At the start: 2 copper layers, 147.2 x 133.8 mm, 72 parts, among them SW1 KEY_01, SW10 KEY_10, SW11 KEY_11, SW12 KEY_12, SW13 KEY_13, SW14 KEY_14, SW15 KEY_15, SW16 KEY_16, SW17 KEY_17, SW18 KEY_18, SW19 KEY_19, SW2 KEY_02, SW20 KEY_20, SW21 KEY_21, SW22 KEY_22, SW23 KEY_23, SW24 KEY_24, SW25 KEY_25, SW26 KEY_26, SW27 KEY_27, SW28 KEY_28, SW29 KEY_29, SW3 KEY_03, SW30 KEY_30, SW31 KEY_31, SW32 KEY_32, SW4 KEY_04, SW5 KEY_05, SW6 KEY_06, SW7 KEY_07, SW8 KEY_08, SW9 KEY_09, U1 nice!nano_v2_socket_24pin

Commit message: fix: KC2 X3 발주 차단 해소
- nice!nano 좌/우 전용 풋프린트 추가 및 controller/switch/power 추적성 정리

- switch pad island routing, edge clearance, DRC error/warning 해소

- 좌/우 PCB, DSN/SES, Gerber/Excellon/fabrication zip/render/DRC JSON 갱신
Parts:
- U1: footprint KC2:NiceNanoV2_Socket_24Pin -> KC2:NiceNanoV2_Socket_24Pin_USB_OUT_LEFT
Routing:
- net L_ROW0: track 288.1 -> 150.6 mm, vias 0 -> 1
- net L_ROW1: track 290.2 -> 154.1 mm, vias 0 -> 1
- net L_ROW3: track 337.6 -> 215.0 mm, vias 0 -> 1
- net L_ROW2: track 309.9 -> 195.0 mm, vias 0 -> 1
- net L_ROW4: track 346.9 -> 237.5 mm, vias 0 -> 1
- net L_COL3: track 244.1 -> 175.8 mm, vias 0 -> 4
- net L_COL2: track 255.0 -> 188.1 mm, vias 0 -> 4
- net L_COL5: track 232.6 -> 167.3 mm, vias 0 -> 2
- net L_COL1: track 274.6 -> 215.3 mm, vias 0 -> 3
- net L_COL0: track 283.7 -> 231.3 mm
- net L_COL4: track 229.8 -> 184.0 mm, vias 0 -> 2
- net L_COL6: track 158.7 -> 123.7 mm
- net LK07_D: track 34.0 -> 21.6 mm
- net LK10_D: track 34.0 -> 21.6 mm
- net LK11_D: track 34.0 -> 21.6 mm
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