File: hardware/kicad/draft/x3-v2/autoroute/kc2_left-x3-v2-71-r8.pre-route.kicad_pcb (KiCad board)
At the start: 2 copper layers, 136.3 x 127.8 mm, 67 parts, among them SW1 KEY_01, SW10 KEY_10, SW11 KEY_11, SW12 KEY_12, SW13 KEY_13, SW14 KEY_14, SW15 KEY_15, SW16 KEY_16, SW17 KEY_17, SW18 KEY_18, SW19 KEY_19, SW2 KEY_02, SW20 KEY_20, SW21 KEY_21, SW22 KEY_22, SW23 KEY_23, SW24 KEY_24, SW25 KEY_25, SW26 KEY_26, SW27 KEY_27, SW28 KEY_28, SW29 KEY_29, SW3 KEY_03, SW30 KEY_30, SW31 KEY_31, SW32 KEY_32, SW4 KEY_04, SW5 KEY_05, SW6 KEY_06, SW7 KEY_07, SW8 KEY_08, SW9 KEY_09, U1 nice!nano_v2_socket_24pin

Commit message: feat(hardware): implement recessed 71-key X3 V2 PCB
Routing:
- net L_COL5: track 144.5 -> 267.0 mm, vias 1 -> 0
- net L_COL2: track 183.6 -> 301.8 mm, vias 3 -> 0
- net L_COL4: track 162.0 -> 277.8 mm, vias 3 -> 0
- net L_COL3: track 179.7 -> 291.1 mm, vias 3 -> 0
- net L_COL1: track 217.9 -> 317.7 mm, vias 4 -> 0
- net L_COL0: track 235.7 -> 300.3 mm, vias 1 -> 0
- net L_COL6: track 110.4 -> 135.3 mm
- net LK01_D: track 13.5 -> 37.5 mm
- net LK14_D: track 13.8 -> 37.5 mm
- net LK20_D: track 13.9 -> 37.5 mm
- net LK27_D: track 13.9 -> 37.5 mm
- net LK08_D: track 14.6 -> 37.5 mm
- net L_ROW4: track 224.8 -> 247.0 mm, vias 1 -> 0
- net L_ROW1: track 150.1 -> 171.3 mm, vias 2 -> 0
- net L_ROW3: track 210.6 -> 229.5 mm, vias 2 -> 0
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