File: hardware/kicad/draft/x3-v2/autoroute/kc2_right-x3-v2-71-r8.pre-route.kicad_pcb (KiCad board)
At the start: 2 copper layers, 164.9 x 127.8 mm, 81 parts, among them SW1 KEY_01, SW10 KEY_10, SW11 KEY_11, SW12 KEY_12, SW13 KEY_13, SW14 KEY_14, SW15 KEY_15, SW16 KEY_16, SW17 KEY_17, SW18 KEY_18, SW19 KEY_19, SW2 KEY_02, SW20 KEY_20, SW21 KEY_21, SW22 KEY_22, SW23 KEY_23, SW24 KEY_24, SW25 KEY_25, SW26 KEY_26, SW27 KEY_27, SW28 KEY_28, SW29 KEY_29, SW3 KEY_03, SW30 KEY_30, SW31 KEY_31, SW32 KEY_32, SW33 KEY_33, SW34 KEY_34, SW35 KEY_35, SW36 KEY_36, SW37 KEY_37, SW38 KEY_38, SW39 KEY_39, SW4 KEY_04, SW5 KEY_05, SW6 KEY_06, SW7 KEY_07, SW8 KEY_08, SW9 KEY_09, U1 nice!nano_v2_socket_24pin

Commit message: feat(hardware): implement recessed 71-key X3 V2 PCB
Routing:
- net R_COL4: track 196.9 -> 430.2 mm, vias 3 -> 0
- net R_COL5: track 233.3 -> 447.6 mm, vias 3 -> 0
- net R_COL6: track 244.5 -> 455.5 mm, vias 4 -> 0
- net R_COL3: track 203.9 -> 412.7 mm, vias 3 -> 0
- net R_COL2: track 180.6 -> 378.7 mm, vias 1 -> 0
- net R_COL1: track 143.6 -> 294.6 mm, vias 2 -> 0
- net R_COL0: track 166.9 -> 259.0 mm
- net RK25_D: track 13.5 -> 37.5 mm
- net RK17_D: track 13.6 -> 37.5 mm
- net RK01_D: track 13.9 -> 37.5 mm
- net RK33_D: track 13.9 -> 37.5 mm
- net RK09_D: track 13.9 -> 37.5 mm
- net R_COL7: track 256.3 -> 278.6 mm, vias 1 -> 0
- net R_ROW2: track 222.5 -> 243.8 mm, vias 3 -> 0
- net R_ROW3: track 236.9 -> 255.2 mm, vias 3 -> 0
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