File: hardware/kicad/draft/x3-v2/kc2_left-x3-v2/kc2_left-x3-v2.kicad_pcb (KiCad board)
At the start: 2 copper layers, 135.1 x 122.5 mm, 76 parts, among them SW1 KEY_01, SW10 KEY_10, SW11 KEY_11, SW12 KEY_12, SW13 KEY_13, SW14 KEY_14, SW15 KEY_15, SW16 KEY_16, SW17 KEY_17, SW18 KEY_18, SW19 KEY_19, SW2 KEY_02, SW20 KEY_20, SW21 KEY_21, SW22 KEY_22, SW23 KEY_23, SW24 KEY_24, SW25 KEY_25, SW26 KEY_26, SW27 KEY_27, SW28 KEY_28, SW29 KEY_29, SW3 KEY_03, SW30 KEY_30, SW31 KEY_31, SW4 KEY_04, SW5 KEY_05, SW6 KEY_06, SW7 KEY_07, SW8 KEY_08, SW9 KEY_09, U1 nice!nano_v2_socket_24pin

Commit message: feat(x3-v2): adopt 1N4148W and dense housing supports
Parts:
- BAT1: value BAT_301230_30x12mm -> 301230_3.7V_100mAh; footprint KC2:BAT_301230_30x12mm -> BAT_301230_30x12mm
- D1, D10, D11, D12, D13, D14, D15, D16, D17, D18, D19, D2, D20, D21, D22, D23, D24, D25, D26, D27, D28, D29, D3, D30, D31, D4, D5, D6, D7, D8, D9: value ES1B_Jingdao_C437840_Eleparts9475342 -> 1N4148W-13-F_DiodesInc_SOD123; footprint D_ES1B_SMA_HandSolder_C437840 -> D_1N4148W_SOD123_HandSolder_DiodesInc
- J_BAT1: value BAT_2Pin_PTH_DirectSolder -> 301230_DIRECT_SOLDER; footprint KC2:BAT_2Pin_PTH_DirectSolder -> BAT_2Pin_PTH_DirectSolder
- SW_PWR1: value SW_IMMS_12V_BSI10_THT -> IMMS-12V_BSI-10; footprint KC2:SW_IMMS_12V_BSI10_THT -> SW_IMMS_12V_BSI10_THT
- moved MH3 0.75 mm to (39.4, 111.0)
- moved MH7 0.50 mm to (165.9, 148.8)
- moved MH8 0.25 mm to (75.2, 134.0)
Routing:
- net L_ROW0: track 145.7 -> 147.6 mm
Other:
- board text added: "Diode: Diodes Inc 1N4148W-13-F SOD-123; pad 1 = row cathode"
- board text removed: "Diode: Jingdao ES1B / C437840 / Eleparts 9475342; pad 1 = row cathode"
